Commit message: Fix robot spawn, arm attachment, wheel physics and gripper meshes

File: src/pickplace_rl_mobile/urdf/mobile_ur3.urdf (robot description, URDF)
Before this commit: robot mobile_manipulator, 38 links, 37 joints
Joints:
- removed joint chassis_to_ur3
- added joint chassis_to_arm_base: type fixed, parent chassis_link, child base_link, origin xyz=0.0 0.0 0.1 rpy=0 0 0

Commit message: Fix gripper collision mesh scale

File: src/pickplace_rl_mobile/urdf/mobile_ur3.urdf (robot description, URDF)
Before this commit: robot mobile_manipulator, 38 links, 37 joints
Links:
- link robotiq_arg2f_base_link: geometry collision mesh filename=package://robotiq_2f_85_gripper_visualization/meshes/collis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 scale=0.001 0.001 0.001; visual mesh filename=package://robotiq_2f_85_gripper_visualization/meshes/visual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 scale=0.001 0.001 0.001

Commit message: Implement rigorous curriculum RL phases, passive casters, and static camera

File: src/pickplace_rl_mobile/urdf/mobile_ur3.urdf (robot description, URDF)
Before this commit: robot mobile_manipulator, 38 links, 37 joints
Links:
- removed link camera_head_color_frame
- removed link camera_head_color_optical_frame
- removed link camera_head_depth_frame
- removed link camera_head_depth_optical_frame
- removed link camera_head_infra1_frame
- removed link camera_head_infra1_optical_frame
- removed link camera_head_infra2_frame
- removed link camera_head_infra2_optical_frame
- removed link camera_head_link
- removed link torso_link
- added link front_caster, mass 0.5; collision sphere radius=0.08; visual sphere radius=0.08
- added link rear_caster, mass 0.5; collision sphere radius=0.08; visual sphere radius=0.08
Joints:
- removed joint base_link_to_torso_link
- removed joint camera_head_color_joint
- removed joint camera_head_color_optical_joint
- removed joint camera_head_depth_joint
- removed joint camera_head_depth_optical_joint
- removed joint camera_head_infra1_joint
- removed joint camera_head_infra1_optical_joint
- removed joint camera_head_infra2_joint
- removed joint camera_head_infra2_optical_joint
- removed joint camera_head_joint
- added joint front_caster_joint: type fixed, parent chassis_link, child front_caster, origin xyz=0.35 0 0 rpy=0 0 0
- added joint rear_caster_joint: type fixed, parent chassis_link, child rear_caster, origin xyz=-0.15 0 0 rpy=0 0 0

Commit message: Fix display URDF path, resize and reposition caster wheels properly

File: src/pickplace_rl_mobile/urdf/mobile_ur3.urdf (robot description, URDF)
Before this commit: robot mobile_manipulator, 30 links, 29 joints
Links:
- link front_caster: mass 0.5 -> 0.2; geometry collision sphere radius=0.04; visual sphere radius=0.04
- link rear_caster: mass 0.5 -> 0.2; geometry collision sphere radius=0.04; visual sphere radius=0.04
Joints:
- joint front_caster_joint: origin xyz=0.35 0 0 rpy=0 0 0 -> xyz=0.20 0 -0.04 rpy=0 0 0
- joint rear_caster_joint: origin xyz=-0.15 0 0 rpy=0 0 0 -> xyz=-0.20 0 -0.04 rpy=0 0 0

Commit message: Cylindrical pickup object, heavier chassis, tipping penalty, RL curriculum README

File: src/pickplace_rl_mobile/urdf/mobile_ur3.urdf (robot description, URDF)
Before this commit: robot mobile_manipulator, 30 links, 29 joints
Links:
- link chassis_link: mass 5.0 -> 10.0

Commit message: Extend front caster to 30cm, penalize arm extension while driving

File: src/pickplace_rl_mobile/urdf/mobile_ur3.urdf (robot description, URDF)
Before this commit: robot mobile_manipulator, 30 links, 29 joints
Joints:
- joint front_caster_joint: origin xyz=0.20 0 -0.04 rpy=0 0 0 -> xyz=0.30 0 -0.04 rpy=0 0 0

Commit message: Scripted pre-grasp, SAC→TQC, heavy chassis, extended casters

File: src/pickplace_rl_mobile/urdf/mobile_ur3.urdf (robot description, URDF)
Before this commit: robot mobile_manipulator, 30 links, 29 joints
Links:
- link chassis_link: mass 10.0 -> 30.0
- link front_caster: mass 0.2 -> 0.5; geometry collision sphere radius=0.06; visual sphere radius=0.06
- link rear_caster: mass 0.2 -> 0.5; geometry collision sphere radius=0.06; visual sphere radius=0.06
Joints:
- joint front_caster_joint: origin xyz=0.30 0 -0.04 rpy=0 0 0 -> xyz=0.22 0 -0.02 rpy=0 0 0
- joint rear_caster_joint: origin xyz=-0.20 0 -0.04 rpy=0 0 0 -> xyz=-0.20 0 -0.02 rpy=0 0 0

Commit message: 60kg chassis, front caster x=30cm, arm folds back during pregrasp

File: src/pickplace_rl_mobile/urdf/mobile_ur3.urdf (robot description, URDF)
Before this commit: robot mobile_manipulator, 30 links, 29 joints
Links:
- link chassis_link: mass 30.0 -> 60.0
Joints:
- joint front_caster_joint: origin xyz=0.22 0 -0.02 rpy=0 0 0 -> xyz=0.30 0 -0.02 rpy=0 0 0

Commit message: Move front caster to x=0.18m, lock base phases 1-3

File: src/pickplace_rl_mobile/urdf/mobile_ur3.urdf (robot description, URDF)
Before this commit: robot mobile_manipulator, 30 links, 29 joints
Joints:
- joint front_caster_joint: origin xyz=0.30 0 -0.02 rpy=0 0 0 -> xyz=0.18 0 -0.02 rpy=0 0 0

Commit message: fix gripper mimic

File: src/pickplace_rl_mobile/urdf/mobile_ur3.urdf (robot description, URDF)
Before this commit: robot mobile_manipulator, 30 links, 29 joints
Joints:
- joint right_outer_knuckle_joint: mimic joint=finger_joint multiplier=-1 offset=0 -> joint=finger_joint multiplier=1 offset=0

Commit message: Fix gripper mimic and mesh materials

File: src/pickplace_rl_mobile/urdf/mobile_ur3.urdf (robot description, URDF)
Before this commit: robot mobile_manipulator, 30 links, 29 joints
Joints:
- joint right_outer_knuckle_joint: mimic joint=finger_joint multiplier=1 offset=0 -> joint=finger_joint multiplier=-1 offset=0

Commit message: update urdf and mtc components

File: src/pickplace_rl_mobile/urdf/mobile_ur3.urdf (robot description, URDF)
Before this commit: robot mobile_manipulator, 30 links, 29 joints
Joints:
- joint right_outer_knuckle_joint: limit lower=0 upper=0.81 effort=1000 velocity=2.0 -> lower=-0.81 upper=0 effort=1000 velocity=2.0

Commit message: fix base link collision scale

File: src/pickplace_rl_mobile/urdf/mobile_ur3.urdf (robot description, URDF)
Before this commit: robot mobile_manipulator, 30 links, 29 joints
Links:
- link robotiq_arg2f_base_link: geometry collision mesh filename=package://robotiq_2f_85_gripper_visualization/meshes/collis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; visual mesh filename=package://robotiq_2f_85_gripper_visualization/meshes/visual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 scale=0.001 0.001 0.001
