Commit message: Fix Robotiq mimic joint, add WBC Gazebo launch, update results

File: src/pickplace_rl_mobile/urdf/mobile_ur3.urdf (robot description, URDF)
Before this commit: robot mobile_manipulator, 30 links, 29 joints
Joints:
- joint right_outer_knuckle_joint: limit lower=-0.81 upper=0 effort=1000 velocity=2.0 -> lower=0 upper=0.81 effort=1000 velocity=2.0; mimic joint=finger_joint multiplier=-1 offset=0 -> joint=finger_joint multiplier=1 offset=0

Commit message: Add Gazebo pick and place images

File: src/pickplace_rl_mobile/urdf/mobile_ur3.urdf (robot description, URDF)
Before this commit: robot mobile_manipulator, 30 links, 29 joints
Links:
- link robotiq_arg2f_base_link: geometry collision mesh filename=package://robotiq_2f_85_gripper_visualization/meshes/collis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; visual mesh filename=package://robotiq_2f_85_gripper_visualization/meshes/collis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

Commit message: Add gripper pad friction

File: src/pickplace_rl_mobile/urdf/mobile_ur3.urdf (robot description, URDF)
Before this commit: robot mobile_manipulator, 30 links, 29 joints
Joints:
- joint finger_joint: limit lower=0 upper=0.8 effort=1000 velocity=2.0 -> lower=0 upper=0.8 effort=20 velocity=2.0
- joint right_outer_knuckle_joint: limit lower=0 upper=0.81 effort=1000 velocity=2.0 -> lower=0 upper=0.81 effort=20 velocity=2.0

File: src/robotiq_2f_85_gripper_visualization/urdf/robotiq_arg2f.xacro (robot description, xacro)
@@ -24,5 +24,5 @@
       </collision>
     </link>
-    <gazebo reference="robotiq_arg2f_base_link">
+    <gazebo reference="${prefix}robotiq_arg2f_base_link">
   <disableFixedJointLumping>true</disableFixedJointLumping>
 </gazebo>

File: src/robotiq_2f_85_gripper_visualization/urdf/robotiq_arg2f_85_model_macro.xacro (robot description, xacro)
@@ -120,4 +120,9 @@
       </collision>
     </link>
+    <!-- Grippy rubber pads: unset friction fell back to the simulator default and the cube slipped out -->
+    <gazebo reference="${prefix}${fingerprefix}_inner_finger_pad">
+      <mu1>2.0</mu1>
+      <mu2>2.0</mu2>
+    </gazebo>
   </xacro:macro>
   <xacro:macro name="outer_finger_joint" params="prefix fingerprefix">
@@ -165,5 +170,5 @@
       <child link="${prefix}left_outer_knuckle" />
       <axis xyz="1 0 0" />
-      <limit lower="0" upper="0.8" velocity="2.0" effort="1000" />
+      <limit lower="0" upper="0.8" velocity="2.0" effort="20" />
     </joint>
     <xacro:finger_joints prefix="${prefix}" fingerprefix="left" reflect="1.0"/>
@@ -175,5 +180,5 @@
       <child link="${prefix}right_outer_knuckle" />
       <axis xyz="1 0 0" />
-      <limit lower="0" upper="0.81" velocity="2.0" effort="1000" />
+      <limit lower="0" upper="0.81" velocity="2.0" effort="20" />
       <mimic joint="${prefix}finger_joint" multiplier="1" offset="0" />
     </joint>
