Commit message: remove hardcoded absolute mesh paths

File: src/moveit_config/config/ur.urdf (robot description, URDF)
Before this commit: robot ur, 34 links, 33 joints
Links:
- link camera_head_link: geometry collision box size=0.02505 0.09 0.025; visual mesh filename=package://ur_description/meshes/d435/visual/d435.stl

File: src/ur_description/urdf/ur.urdf (robot description, URDF)
Before this commit: robot ur, 34 links, 33 joints
Links:
- link camera_head_link: geometry collision box size=0.02505 0.09 0.025; visual mesh filename=package://ur_description/meshes/d435/visual/d435.stl

File: src/ur_description/urdf/ur_robot.urdf (robot description, URDF)
Before this commit: robot ur, 34 links, 33 joints
Links:
- link camera_head_link: geometry collision box size=0.02505 0.09 0.025; visual mesh filename=package://ur_description/meshes/d435/visual/d435.stl

File: src/ur_robot.urdf (robot description, URDF)
Before this commit: robot ur, 34 links, 33 joints
Links:
- link camera_head_link: geometry collision box size=0.02505 0.09 0.025; visual mesh filename=package://ur_description/meshes/d435/visual/d435.stl
